File: pcb/Dormo/Dormo.kicad_pcb (KiCad board)
At the start: 4 copper layers, 229 x 39 mm, 120 parts, among them J2 USB_C_Receptacle_USB2.0_16P, J3 FPC, 6P, P=0.5mm, J4 Conn_01x02, Q1 AO3401A, U1 ESP32-C3, U2 MIC5504-3.3YM5, U3 BRCL4054BME, Y1 40MHz

Commit message: minor layout tweaks
Parts:
- moved C30 88.4 mm to (157.6, 137.4)
- moved D18 88.4 mm to (164.6, 133.4)
- moved R31 88.4 mm to (160.7, 133.4)
- moved SW17 88.4 mm to (162.5, 137.5)
- moved SW1 81.7 mm to (137.5, 127.5)
- moved C24 80.5 mm to (122.6, 139.9)
- moved D12 80.5 mm to (129.6, 135.9)
- moved R25 80.5 mm to (125.7, 135.9)
- moved SW11 80.5 mm to (127.5, 140.0)
- moved C33 74.2 mm to (182.6, 114.9)
- moved C34 74.2 mm to (182.6, 139.9)
- moved D21 74.2 mm to (189.6, 110.9)
- moved D22 74.2 mm to (189.6, 135.9)
- moved R34 74.2 mm to (185.7, 110.9)
- moved R35 74.2 mm to (185.7, 135.9)
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Other:
- board size 229 x 39 mm -> 150 x 45 mm
- board text added: "Centerline"
- board text added: "Target size: approx 150mm x 45mm"
- board text removed: "Target size: approx 45mm x 150 mm"

Commit message: first pass of PCB routing
Parts:
- added JP2: Bridged, Jumper:SolderJumper-2_P1.3mm_Bridged_RoundedPad1.0x1.5mm, F.Cu at (80.5, 135.5)
- moved C9 34.8 mm to (77.5, 142.3), turned to -90 degrees
- moved R10 33.0 mm to (75.5, 142.3), turned to -90 degrees
- moved R9 31.1 mm to (77.5, 138.7), turned to -90 degrees
- moved R6 30.2 mm to (60.2, 118.6), turned to -90 degrees
- moved D2 29.0 mm to (75.5, 138.6), turned to -90 degrees
- moved R5 26.5 mm to (64.0, 118.6), turned to -90 degrees
- moved R11 25.9 mm to (62.0, 118.6), turned to -90 degrees
- moved C13 23.5 mm to (70.0, 111.2), turned to 90 degrees
- moved R13 21.2 mm to (80.5, 133.2)
- moved D3 19.9 mm to (76.3, 135.5), turned to 180 degrees
- moved C11 17.7 mm to (79.2, 120.2), turned to 0 degrees
- moved R12 14.5 mm to (76.3, 133.5), turned to 0 degrees
- moved C10 12.6 mm to (77.7, 109.2)
- moved U1 10.8 mm to (73.8, 118.0)
- moved C4 9.77 mm to (73.5, 106.5), turned to 0 degrees
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Connections:
- D1 pad 1: /LATCH -> /LATCH_MX
- D10 pad 1: /LATCH -> /LATCH_MX
- D11 pad 1: /LATCH -> /LATCH_MX
- D12 pad 1: /LATCH -> /LATCH_MX
- D13 pad 1: /LATCH -> /LATCH_MX
- D14 pad 1: /LATCH -> /LATCH_MX
- D15 pad 1: /LATCH -> /LATCH_MX
- D16 pad 1: /LATCH -> /LATCH_MX
- D17 pad 1: /LATCH -> /LATCH_MX
- D18 pad 1: /LATCH -> /LATCH_MX
- D19 pad 1: /LATCH -> /LATCH_MX
- D20 pad 1: /LATCH -> /LATCH_MX
- D21 pad 1: /LATCH -> /LATCH_MX
- D22 pad 1: /LATCH -> /LATCH_MX
- D4 pad 1: /LATCH -> /LATCH_MX
- D5 pad 1: /LATCH -> /LATCH_MX
- D6 pad 1: /LATCH -> /LATCH_MX
- D7 pad 1: /LATCH -> /LATCH_MX
- D8 pad 1: /LATCH -> /LATCH_MX
- D9 pad 1: /LATCH -> /LATCH_MX
- R9 pad 1: /LATCH -> Net-(R9-Pad1)
- SW1 pad 1: /LATCH -> Net-(R9-Pad1)
Routing:
- net /LATCH_MX: track 0.00 -> 339.1 mm, vias 0 -> 21
- net /COL_3: track 0.00 -> 179.6 mm, vias 0 -> 8
- net /GPIO15: track 0.00 -> 170.0 mm, vias 0 -> 4
- net /COL_4: track 0.00 -> 145.7 mm, vias 0 -> 4
- net /COL_1: track 0.00 -> 143.6 mm, vias 0 -> 12
- net /GPIO14: track 0.00 -> 126.1 mm, vias 0 -> 6
- net /COL_2: track 0.00 -> 123.4 mm, vias 0 -> 10
- net /+VBAT: track 0.00 -> 121.5 mm, vias 0 -> 4
- net /GPIO13: track 0.00 -> 106.5 mm, vias 0 -> 6
- net /GPIO12: track 0.00 -> 100.2 mm, vias 0 -> 4
- net Net-(R9-Pad1): track 0.00 -> 83.3 mm, vias 0 -> 4
- net /GPIO10: track 0.00 -> 74.3 mm, vias 0 -> 2
- net /BTN: track 0.00 -> 47.4 mm, vias 0 -> 2
- net /GPIO19: track 0.00 -> 45.2 mm, vias 0 -> 2
- net /GPIO18: track 0.00 -> 44.0 mm, vias 0 -> 2
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- added copper zone on F.Cu, net /+3V3
- added copper zone on In1.Cu, net /+3V3
- added copper zone on F.Cu, net /+VBAT
- added copper zone on F.Cu, net /+VUSB
- added copper zone on B.Cu, net GND
- added copper zone on F.Cu, net GND
- added copper zone on In2.Cu, net GND

Commit message: minor adjustements
Parts:
- moved R7 1.64 mm to (62.8, 140.8)
- moved R8 1.64 mm to (62.8, 143.5)
Routing:
- net Net-(J2-CC2): track 4.45 -> 5.73 mm
- net Net-(J2-CC1): track 4.53 -> 5.63 mm
- net /GPIO18: track 44.0 -> 43.0 mm
- net /GPIO19: track 45.2 -> 44.3 mm
Other:
- outline, holes or cut-outs redrawn
Changed lines of the file:
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@@
 	(footprint "Resistor_SMD:R_0603_1608Metric_Pad0.98x0.95mm_HandSolder"
 		(layer "F.Cu")
-		(at 62.0875 145 180)
+		(at 62.75 143.5 180)
 		(descr "Resistor SMD 0603 (1608 Metric), square (rectangular) end terminal, IPC-7351 nominal with elongated pad for handsoldering. (Body size source: IPC-SM-782 page 72, https://www.pcb-3d.com/wordpress/wp-content/uploads/ipc-sm-782a_amendment_1_and_2.pdf), generated with kicad-footprint-generator")
 		(tags "resistor handsolder")
@@
 	(footprint "Resistor_SMD:R_0603_1608Metric_Pad0.98x0.95mm_HandSolder"
 		(layer "F.Cu")
-		(at 62.0875 142.25)
+		(at 62.75 140.75)
 		(descr "Resistor SMD 0603 (1608 Metric), square (rectangular) end terminal, IPC-7351 nominal with elongated pad for handsoldering. (Body size source: IPC-SM-782 page 72, https://www.pcb-3d.com/wordpress/wp-content/uploads/ipc-sm-782a_amendment_1_and_2.pdf), generated with kicad-footprint-generator")
 		(tags "resistor handsolder")
@@
 		)
 	)
+	(gr_rect
+		(start 48.8 103.8)
+		(end 61.3 113.3)
+		(stroke
+			(width 0.1)
+			(type solid)
+		)
+		(fill yes)
+		(layer "F.Mask")
+	)
+	(gr_rect
+		(start 49.2 104.4)
+		(end 61.3 113.3)
+		(stroke
+			(width 0.1)
+			(type solid)
+		)
+		(fill yes)
+		(layer "B.Mask")
+	)
+	(gr_line
+		(start 62.75 148)
+		(end 62.75 107)
+		(stroke
+			(width 0.1)
+			(type default)
+		)
+		(layer "Cmts.User")
+	)
 	(gr_line
 		(start 172.5 127.5)
@@
 		(layer "Cmts.User")
 	)
+	(gr_arc
+		(start 64.75 106)
+		(mid 62.75 108)
+		(end 60.75 106)
+		(stroke
+			(width 0.05)
+			(type default)
+		)
+		(layer "Edge.Cuts")
+	)
 	(gr_line
-		(start 200 105)
-		(end 200 150)
+		(start 60.75 150)
+		(end 52.5 150)
+		(stroke
+			(width 0.05)
+			(type default)
+		)
+		(layer "Edge.Cuts")
+	)
+	(gr_arc
+		(start 50 107.5)
+		(mid 50.732233 105.732233)
+		(end 52.5 105)
 		(stroke
 			(width 0.05)
@@
 	)
 	(gr_line
-		(start 50 150)
-		(end 50 105)
+		(start 200 107.5)
+		(end 200 147.5)
+		(stroke
+			(width 0.05)
+			(type default)
+		)
+		(layer "Edge.Cuts")
+	)
+	(gr_arc
+		(start 197.5 105)
+		(mid 199.267767 105.732233)
+		(end 200 107.5)
 		(stroke
 			(width 0.05)
@@
 	)
 	(gr_line
-		(start 50 105)
-		(end 200 105)
+		(start 64.75 105)
+		(end 64.75 106)
+		(stroke
+			(width 0.05)
+			(type default)
+		)
+		(layer "Edge.Cuts")
+	)
+	(gr_arc
+		(start 52.5 150)
+		(mid 50.732233 149.267767)
+		(end 50 147.5)
 		(stroke
 			(width 0.05)
@@
 	)
 	(gr_line
-		(start 200 150)
-		(end 50 150)
+		(start 60.75 149)
+		(end 60.75 150)
+		(stroke
+			(width 0.05)
+			(type default)
+		)
+		(layer "Edge.Cuts")
+	)
+	(gr_line
+		(start 50 147.5)
+		(end 50 107.5)
+		(stroke
+			(width 0.05)
+			(type default)
+		)
+		(layer "Edge.Cuts")
+	)
+	(gr_arc
+		(start 200 147.5)
+		(mid 199.267767 149.267767)
+		(end 197.5 150)
+		(stroke
+			(width 0.05)
+			(type default)
+		)
+		(layer "Edge.Cuts")
+	)
+	(gr_line
+		(start 64.75 105)
+		(end 197.5 105)
+		(stroke
+			(width 0.05)
+			(type default)
+		)
+		(layer "Edge.Cuts")
+	)
+	(gr_line
+		(start 64.75 149)
+		(end 64.75 150)
+		(stroke
+			(width 0.05)
+			(type default)
+		)
+		(layer "Edge.Cuts")
+	)
+	(gr_line
+		(start 60.75 105)
+		(end 60.75 106)
+		(stroke
+			(width 0.05)
+			(type default)
+		)
+		(layer "Edge.Cuts")
+	)
+	(gr_line
+		(start 60.75 105)
+		(end 52.5 105)
+		(stroke
+			(width 0.05)
+			(type default)
+		)
+		(layer "Edge.Cuts")
+	)
+	(gr_line
+		(start 197.5 150)
+		(end 64.75 150)
+		(stroke
+			(width 0.05)
+			(type default)
+		)
+		(layer "Edge.Cuts")
+	)
+	(gr_arc
+		(start 60.75 149)
+		(mid 62.75 147)
+		(end 64.75 149)
 		(stroke
 			(width 0.05)
@@
 	)
 	(segment
-		(start 57.574 144.18)
-		(end 56.8 144.18)
+		(start 66 141)
+		(end 64.5 142.5)
 		(width 0.15)
 		(layer "F.Cu")
@@
 	)
 	(segment
-		(start 57.696 144.058)
-		(end 57.574 144.18)
+		(start 57.574 144.18)
+		(end 56.8 144.18)
 		(width 0.15)
 		(layer "F.Cu")
@@
 	)
 	(segment
-		(start 58.492 143.6)
-		(end 58.146 143.254)
+		(start 57.696 144.058)
+		(end 57.574 144.18)
 		(width 0.15)
 		(layer "F.Cu")
@@
 	)
 	(segment
-		(start 66 142)
-		(end 64.4 143.6)
+		(start 58.9 142.5)
+		(end 58.146 143.254)
 		(width 0.15)
 		(layer "F.Cu")
@@
 	)
 	(segment
-		(start 64.4 143.6)
-		(end 58.492 143.6)
+		(start 57.622 143.18)
+		(end 57.696 143.254)
 		(width 0.15)
 		(layer "F.Cu")
@@
 	)
 	(segment
-		(start 58.146 143.254)
-		(end 57.696 143.254)
+		(start 64.5 142.5)
+		(end 58.9 142.5)
 		(width 0.15)
 		(layer "F.Cu")
@@
 	)
 	(segment
-		(start 57.622 143.18)
+		(start 58.146 143.254)
 		(end 57.696 143.254)
 		(width 0.15)
@@
 	(segment
 		(start 66 140.8)
-		(end 66 142)
+		(end 66 141)
 		(width 0.15)
 		(layer "F.Cu")
@@
 	)
 	(segment
-		(start 60.995 145.18)
-		(end 61.175 145)
+		(start 59.25 143.75)
+		(end 61.5875 143.75)
 		(width 0.2)
 		(layer "F.Cu")
@@
 	(segment
 		(start 56.8 145.18)
-		(end 60.995 145.18)
+		(end 57.82 145.18)
 		(width 0.2)
 		(layer "F.Cu")
@@
 	)
 	(segment
-		(start 65.2 142)
-		(end 64.199 143.001)
-		(width 0.15)
+		(start 57.82 145.18)
+		(end 59.25 143.75)
+		(width 0.2)
 		(layer "F.Cu")
-		(net 48)
+		(net 46)
 	)
 	(segment
-		(start 58.389388 143.001)
-		(end 58.142388 142.754)
-		(width 0.15)
+		(start 61.5875 143.75)
+		(end 61.8375 143.5)
+		(width 0.2)
 		(layer "F.Cu")
-		(net 48)
+		(net 46)
 	)
 	(segment
-		(start 66.3 139.5)
-		(end 65.2 140.6)
+		(start 64.05 141.75)
+		(end 59.146388 141.75)
 		(width 0.15)
 		(layer "F.Cu")
@@
 	)
 	(segment
-		(start 56.8 143.68)
-		(end 55.978 143.68)
+		(start 56.874 142.754)
+		(end 56.8 142.68)
 		(width 0.15)
 		(layer "F.Cu")
@@
 	)
 	(segment
-		(start 75.55 115.004988)
-		(end 75.736658 114.81833)
+		(start 58.142388 142.754)
+		(end 56.874 142.754)
 		(width 0.15)
 		(layer "F.Cu")
@@
 	)
 	(segment
-		(start 75.55 115.55)
-		(end 75.55 115.004988)
+		(start 56.8 143.68)
+		(end 55.978 143.68)
 		(width 0.15)
 		(layer "F.Cu")
@@
 	)
 	(segment
-		(start 56.874 142.754)
-		(end 56.8 142.68)
+		(start 75.55 115.004988)
+		(end 75.736658 114.81833)
 		(width 0.15)
 		(layer "F.Cu")
@@
 	)
 	(segment
-		(start 65.2 140.6)
-		(end 65.2 142)
+		(start 75.55 115.55)
+		(end 75.55 115.004988)
 		(width 0.15)
 		(layer "F.Cu")
@@
 	)
 	(segment
-		(start 64.199 143.001)
-		(end 58.389388 143.001)
+		(start 59.146388 141.75)
+		(end 58.142388 142.754)
 		(width 0.15)
 		(layer "F.Cu")
@@
 	)
 	(segment
-		(start 55.904 143.606)
-		(end 55.904 142.754)
+		(start 66.3 139.5)
+		(end 64.05 141.75)
 		(width 0.15)
 		(layer "F.Cu")
@@
 	)
 	(segment
-		(start 58.142388 142.754)
-		(end 56.874 142.754)
+		(start 55.904 143.606)
+		(end 55.904 142.754)
 		(width 0.15)
 		(layer "F.Cu")
@@
 	)
 	(segment
-		(start 57.87 142.378)
-		(end 58.298132 142.378)
+		(start 59.25 140.75)
+		(end 61.8375 140.75)
 		(width 0.2)
 		(layer "F.Cu")
@@
 	)
 	(segment
-		(start 61.025 142.4)
-		(end 61.175 142.25)
+		(start 57.82 142.18)
+		(end 59.25 140.75)
 		(width 0.2)
 		(layer "F.Cu")
@@
 	(segment
 		(start 56.8 142.18)
-		(end 57.672 142.18)
-		(width 0.2)
-		(layer "F.Cu")
-		(net 50)
-	)
-	(segment
-		(start 58.298132 142.378)
-		(end 58.320132 142.4)
-		(width 0.2)
-		(layer "F.Cu")
-		(net 50)
-	)
-	(segment
-		(start 57.672 142.18)
-		(end 57.87 142.378)
-		(width 0.2)
-		(layer "F.Cu")
-		(net 50)
-	)
-	(segment
-		(start 58.320132 142.4)
-		(end 61.025 142.4)
+		(end 57.82 142.18)
 		(width 0.2)
 		(layer "F.Cu")
@@
 		(min_thickness 0.25)
 		(filled_areas_thickness no)
-		(fill
+		(fill yes
 			(thermal_gap 0.5)
 			(thermal_bridge_width 0.5)
@@
 		(net 0)
 		(net_name "")
-		(layers "F.Cu" "F.Mask" "B.Cu" "B.Mask" "In1.Cu" "In2.Cu")
+		(layers "F.Cu" "B.Cu" "In1.Cu" "In2.Cu")
 		(hatch edge 0.5)
 		(connect_pads
@@
 		(keepout
 			(tracks allowed)
-			(vias not_allowed)
-			(pads not_allowed)
-			(copperpour allowed)
+			(vias allowed)
+			(pads allowed)
+			(copperpour not_allowed)
 			(footprints allowed)
 		)
